File: ursinia.kicad_pcb (KiCad board)
At the start: 2 copper layers, 70.7 x 53.3 mm, 13 parts, among them J1 NEIGHBOR1, J2 NEIGHBOR2, J7 BONUS_ROW, U1 M24C02-FMN6TP

Commit message: complete design
Parts:
- added J10: GROVE-CONNECTOR-DIP_4P-2.0_, OPL_Connectors:HW4-2.0, F.Cu at (139.1, 84.2)
- added J11: GROVE-CONNECTOR-DIP_4P-2.0_, OPL_Connectors:HW4-2.0, F.Cu at (150.1, 84.2)
- added J12: GROVE-CONNECTOR-DIP_4P-2.0_, OPL_Connectors:HW4-2.0, F.Cu at (161.1, 84.2)
- added J13: GROVE-CONNECTOR-DIP_4P-2.0_, OPL_Connectors:HW4-2.0-90D, F.Cu at (173.1, 84.2)
- added J14: GROVE-CONNECTOR-DIP_4P-2.0_, OPL_Connectors:HW4-2.0, F.Cu at (139.1, 106.2)
- added J15: GROVE-CONNECTOR-DIP_4P-2.0_, OPL_Connectors:HW4-2.0, F.Cu at (150.1, 106.2)
- added J16: GROVE-CONNECTOR-DIP_4P-2.0_, OPL_Connectors:HW4-2.0, F.Cu at (161.1, 106.2)
- added J17: GROVE-CONNECTOR-DIP_4P-2.0_, OPL_Connectors:HW4-2.0-90D, F.Cu at (173.1, 106.2)
- added J3: GROVE-CONNECTOR-DIP_4P-2.0_, OPL_Connectors:HW4-2.0-90D, F.Cu at (115.0, 89.2)
- added J4: GROVE-CONNECTOR-DIP_4P-2.0_, OPL_Connectors:HW4-2.0-90D, F.Cu at (115.0, 101.2)
- added J5: GROVE-CONNECTOR-DIP_4P-2.0_, OPL_Connectors:HW4-2.0, F.Cu at (139.1, 95.2)
- added J6: GROVE-CONNECTOR-DIP_4P-2.0_, OPL_Connectors:HW4-2.0, F.Cu at (150.1, 95.2)
- added J8: GROVE-CONNECTOR-DIP_4P-2.0_, OPL_Connectors:HW4-2.0, F.Cu at (161.1, 95.2)
- added J9: GROVE-CONNECTOR-DIP_4P-2.0_, OPL_Connectors:HW4-2.0-90D, F.Cu at (173.1, 95.2)
- added R2: 2k, Resistor_SMD:R_0603_1608Metric_Pad1.05x0.95mm_HandSolder, B.Cu at (173.8, 102.3)
- added R3: 2k, Resistor_SMD:R_0603_1608Metric_Pad1.05x0.95mm_HandSolder, B.Cu at (173.7, 105.2)
- C1, JP1, JP2, JP3, R1, U1: moved to B.Cu
- moved JP1 18.1 mm to (167.6, 95.0), turned to 90 degrees
- moved JP2 15.3 mm to (165.6, 95.0), turned to 90 degrees
- moved JP3 12.5 mm to (163.6, 95.0), turned to 90 degrees
- moved U1 5.89 mm to (165.6, 88.0), turned to 90 degrees
- moved R1 5.50 mm to (164.6, 82.1), turned to 90 degrees
- moved C1 3.00 mm to (167.6, 82.1), turned to 270 degrees
Routing:
- net /P2_3: track 0.00 -> 67.3 mm
- net /P2_4: track 0.00 -> 65.5 mm
- net /P7_7: track 0.00 -> 42.7 mm
- net /P6_4: track 0.00 -> 35.1 mm
- net /P4_3: track 0.00 -> 35.0 mm
- net /I2C0_SCL: track 16.4 -> 49.5 mm
- net /P6_5: track 0.00 -> 32.5 mm
- net /P2_10: track 0.00 -> 32.5 mm
- net /P5_5: track 0.00 -> 31.3 mm
- net /P2_11: track 0.00 -> 30.6 mm
- net /P5_4: track 0.00 -> 29.9 mm
- net /P9_6: track 0.00 -> 29.7 mm
- net /P1_16: track 0.00 -> 28.9 mm
- net /I2C0_SDA: track 17.8 -> 46.4 mm
- net /P4_5: track 0.00 -> 28.1 mm
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Other:
- net class Default: clearance 0.1524 -> 0.2032
- rule trace_clearance: 0.1524 -> 0.2032
- board text added: "26 September 2019"
- board text added: "ADC0_0"
- board text added: "ADC0_5"
- board text added: "Analog"
- board text added: "Connected Grove modules must be 3.3V compatible."
- board text added: "Digital"
- board text added: "Grove base neighbor for GreatFET"
- board text added: "I2C"
- board text added: "P1_16"
- board text added: "P2_10"
- board text added: "P2_11"
- board text added: "P2_3"
- board text added: "P2_4"
- board text added: "P4_3"
- board text added: "P4_4"
- board text added: "P4_5"
- board text added: "P5_4"
- board text added: "P5_5"
- board text added: "P5_6"
- board text added: "P5_7"
- board text added: "P6_4"
- board text added: "P6_5"
- board text added: "P7_0"
- board text added: "P7_1"
- board text added: "P7_7"
- board text added: "P9_6"
- board text added: "UART"
- board text added: "Ursinia"
- board text removed: "24 September 2019"
- board text removed: "I/O pins are 3.3V."
- board text removed: "My Neighbor"
- board text removed: "for GreatFET"

Commit message: adopt OSHWA convention for SPI signal names https://www.oshwa.org/a-resolution-to-redefine-spi-signal-names
Other:
- board text added: "CIPO"
- board text added: "COPI"
- board text added: "CS"
- board text removed: "MISO"
- board text removed: "MOSI"
- board text removed: "SSEL"
Changed lines of the file:
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@@
     (effects (font (size 0.635 0.508) (thickness 0.1016)) (justify mirror))
   )
-  (gr_text MOSI (at 172.72 119.38) (layer B.SilkS)
-    (effects (font (size 0.635 0.508) (thickness 0.1016)) (justify mirror))
-  )
-  (gr_text MISO (at 172.72 116.84) (layer B.SilkS)
+  (gr_text COPI (at 172.72 119.38) (layer B.SilkS)
+    (effects (font (size 0.635 0.508) (thickness 0.1016)) (justify mirror))
+  )
+  (gr_text CIPO (at 172.72 116.84) (layer B.SilkS)
     (effects (font (size 0.635 0.508) (thickness 0.1016)) (justify mirror))
   )
@@
     (effects (font (size 0.635 0.508) (thickness 0.1016)) (justify mirror))
   )
-  (gr_text SSEL (at 167.64 121.412) (layer B.SilkS)
+  (gr_text CS (at 167.64 121.412) (layer B.SilkS)
     (effects (font (size 0.635 0.508) (thickness 0.1016)) (justify mirror))
   )
@@
     (effects (font (size 0.635 0.508) (thickness 0.1016)))
   )
-  (gr_text SSEL (at 167.64 121.412) (layer F.SilkS)
-    (effects (font (size 0.635 0.508) (thickness 0.1016)))
-  )
-  (gr_text MISO (at 172.72 116.84) (layer F.SilkS)
-    (effects (font (size 0.635 0.508) (thickness 0.1016)))
-  )
-  (gr_text MOSI (at 172.72 119.38) (layer F.SilkS)
-    (effects (font (size 0.635 0.508) (thickness 0.1016)))
-  )
+  (gr_text CS (at 167.64 121.412) (layer F.SilkS)
+    (effects (font (size 0.635 0.508) (thickness 0.1016)))
+  )
+  (gr_text CIPO (at 172.72 116.84) (layer F.SilkS)
+    (effects (font (size 0.635 0.508) (thickness 0.1016)))
+  )
+  (gr_text COPI (at 172.72 119.38) (layer F.SilkS)
+    (effects (font (size 0.635 0.508) (thickness 0.1016)))
+  )
